File: poweramp/poweramp.sch (KiCad schematic (older format))
At the start: 12 parts, among them J1 CONTROL, J2 POWER, J3 LOAD, Q1 BC547, Q2 BC557, Q3 BD179

Commit message: Minor fixes in power amplifier schematic
Parts:
- C1: footprint ~ -> BOX3_1
Connections:
- net +12V: now also J3.2; no longer J3.1
- net at D1.2, Q3.2, R4.2: now also J3.1; no longer J3.2
Changed lines of the file:
@@
 $EndComp
 $Comp
-L GND #PWR3
+L GND #PWR01
 U 1 1 5460E547
 P 4700 3300
-F 0 "#PWR3" H 4700 3300 30  0001 C CNN
+F 0 "#PWR01" H 4700 3300 30  0001 C CNN
 F 1 "GND" H 4700 3230 30  0001 C CNN
 F 2 "" H 4700 3300 60  0000 C CNN
@@
 $EndComp
 $Comp
-L +5V #PWR2
+L +5V #PWR02
 U 1 1 5460E557
 P 4700 3150
-F 0 "#PWR2" H 4700 3240 20  0001 C CNN
+F 0 "#PWR02" H 4700 3240 20  0001 C CNN
 F 1 "+5V" H 4700 3240 30  0000 C CNN
 F 2 "" H 4700 3150 60  0000 C CNN
@@
 	6050 2300 6150 2300
 $Comp
-L +5V #PWR5
+L +5V #PWR03
 U 1 1 5460E9DD
 P 6400 1800
-F 0 "#PWR5" H 6400 1890 20  0001 C CNN
+F 0 "#PWR03" H 6400 1890 20  0001 C CNN
 F 1 "+5V" H 6400 1890 30  0000 C CNN
 F 2 "" H 6400 1800 60  0000 C CNN
@@
 F 0 "C1" H 7050 2200 40  0000 L CNN
 F 1 "100" H 7056 2015 40  0000 L CNN
-F 2 "~" H 7088 1950 30  0000 C CNN
+F 2 "BOX3_1" H 7088 1950 30  0000 C CNN
 F 3 "~" H 7050 2100 60  0000 C CNN
 	1    7050 2100
@@
 	7400 1900 7400 2200
 $Comp
-L +12V #PWR6
+L +12V #PWR04
 U 1 1 5460EC9F
 P 7050 1800
-F 0 "#PWR6" H 7050 1750 20  0001 C CNN
+F 0 "#PWR04" H 7050 1750 20  0001 C CNN
 F 1 "+12V" H 7050 1900 30  0000 C CNN
 F 2 "" H 7050 1800 60  0000 C CNN
@@
 	7050 1800 7050 1900
 $Comp
-L GND #PWR7
+L GND #PWR05
 U 1 1 5460ECC1
 P 7050 3800
-F 0 "#PWR7" H 7050 3800 30  0001 C CNN
+F 0 "#PWR05" H 7050 3800 30  0001 C CNN
 F 1 "GND" H 7050 3730 30  0001 C CNN
 F 2 "" H 7050 3800 60  0000 C CNN
@@
 $EndComp
 $Comp
-L GND #PWR4
+L GND #PWR06
 U 1 1 5460ED83
 P 5100 4150
-F 0 "#PWR4" H 5100 4150 30  0001 C CNN
+F 0 "#PWR06" H 5100 4150 30  0001 C CNN
 F 1 "GND" H 5100 4080 30  0001 C CNN
 F 2 "" H 5100 4150 60  0000 C CNN
@@
 $EndComp
 $Comp
-L +12V #PWR1
+L +12V #PWR07
 U 1 1 5460ED92
 P 4600 4150
-F 0 "#PWR1" H 4600 4100 20  0001 C CNN
+F 0 "#PWR07" H 4600 4100 20  0001 C CNN
 F 1 "+12V" H 4600 4250 30  0000 C CNN
 F 2 "" H 4600 4150 60  0000 C CNN
@@
 L CONN_2 J3
 U 1 1 5460EE05
-P 8150 2450
-F 0 "J3" H 7950 2825 50  0000 L CNN
-F 1 "LOAD" H 7950 2725 50  0000 L CNN
-F 2 "SIP2" H 8150 2450 50  0001 C CNN
-F 3 "~" H 8150 2450 60  0000 C CNN
-	1    8150 2450
-	1    0    0    -1
-$EndComp
-Wire Wire Line
+P 8150 2400
+F 0 "J3" H 7950 2775 50  0000 L CNN
+F 1 "LOAD" H 7950 2675 50  0000 L CNN
+F 2 "SIP2" H 8150 2400 50  0001 C CNN
+F 3 "~" H 8150 2400 60  0000 C CNN
+	1    8150 2400
+	1    0    0    1
+$EndComp
+Wire Wire Line
