File: poweramp/poweramp.sch (KiCad schematic (older format))
At the start: 12 parts, among them J1 CONTROL, J2 POWER, J3 LOAD, Q1 BC547, Q2 BC557, Q3 BD179

Commit message: Replaced a resistor value in the schematic with one I had in my toolbox
Parts:
- R2: value 2k2 -> 3k3
Changed lines of the file:
@@
 Sheet 1 1
 Title ""
-Date "11 nov 2014"
+Date "15 nov 2014"
 Rev ""
 Comp ""
@@
 P 5800 2300
 F 0 "R2" H 5900 2350 50  0000 L CNN
-F 1 "2k2" H 5900 2250 50  0000 L CNN
+F 1 "3k3" H 5900 2250 50  0000 L CNN
 F 2 "AX3_1N" H 5800 2300 50  0001 C CNN
 F 3 "" H 5800 2300 60  0000 C CNN
